File: TinyESP/esp8266_schematic.brd (EAGLE design)
At the start: 100 x 80 mm, 12 parts, among them T1 BTA26-V

Commit message: up1
Parts:
- C1: value (none) -> 100nF
- R1, R2: value (none) -> 1k; device rcl:0204/5 -> rcl:0207/2V
- R3: value (none) -> 1k
- R4, R5: value (none) -> 470
- moved J2 10.2 mm to (24.1, 34.3)
- moved SWITCH1 8.04 mm to (12.2, 27.6)
- moved T1 6.99 mm to (22.9, 26.0)
- moved HLK1 3.18 mm to (53.3, 21.0)
- moved R1 0.64 mm to (12.7, 8.26)
- moved R2 0.63 mm to (12.7, 22.2)
Routing:
- net N$6: track 13.3 -> 0.00 mm
- net BOMB: track 21.9 -> 11.7 mm
- net N$3: track 24.2 -> 14.7 mm, vias 0 -> 1
- net GND: track 87.4 -> 78.2 mm
- net +3V3: track 62.0 -> 54.8 mm
- net NEUTRAL: track 26.5 -> 24.7 mm
- net N$2: track 9.42 -> 7.67 mm
- net LINE: track 40.4 -> 39.5 mm
Other:
- board size 100 x 80 mm -> 55.5 x 35.6 mm

Commit message: up2
Connections:
- removed net N$2: R1.2, SV1.6
- net TRIAC: now also R1.2, SV1.6
Routing:
- net TRIAC: track 0.00 -> 7.67 mm
- net N$2: track 7.67 -> 0.00 mm
Changed lines of the file:
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@@
 </elements>
 <signals>
-<signal name="N$2">
-<contactref element="SV1" pad="6"/>
-<contactref element="R1" pad="2"/>
-<wire x1="13.97" y1="8.255" x2="15.875" y2="10.16" width="0.508" layer="16"/>
-<wire x1="15.875" y1="10.16" x2="15.875" y2="12.7" width="0.508" layer="16"/>
-<wire x1="15.875" y1="12.7" x2="14.605" y2="13.97" width="0.508" layer="16"/>
-<wire x1="14.605" y1="13.97" x2="13.97" y2="13.97" width="0.508" layer="16"/>
-</signal>
 <signal name="N$3">
 <contactref element="SV1" pad="4"/>
@@
 <signal name="TRIAC">
 <contactref element="OK1" pad="1"/>
+<contactref element="SV1" pad="6"/>
+<contactref element="R1" pad="2"/>
+<wire x1="13.97" y1="8.255" x2="15.875" y2="10.16" width="0.508" layer="16"/>
+<wire x1="15.875" y1="10.16" x2="15.875" y2="12.7" width="0.508" layer="16"/>
+<wire x1="15.875" y1="12.7" x2="14.605" y2="13.97" width="0.508" layer="16"/>
+<wire x1="14.605" y1="13.97" x2="13.97" y2="13.97" width="0.508" layer="16"/>
+<wire x1="15.875" y1="12.7" x2="39.37" y2="13.97" width="0" layer="19" extent="16-16"/>
 </signal>
 <signal name="N$4">
