File: TinyESP/esp8266_schematic.sch (EAGLE design)
At the start: 12 parts, among them T1 BTA26-V

Commit message: up1
Parts:
- C1: value (none) -> 100nF
- R1, R2: value (none) -> 1k; device rcl:R-EU_0204/5 -> rcl:R-US_0207/2V
- R3: value (none) -> 1k
- R4, R5: value (none) -> 470
Other:
- moved on the sheet: T1
Changed lines of the file:
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@@
 <part name="HLK1" library="HLK-PM01" deviceset="HLK-PM01" device="3W"/>
 <part name="T1" library="triac" library_urn="urn:adsk.eagle:library:403" deviceset="BTA26" device="-V" package3d_urn="urn:adsk.eagle:package:30155/1"/>
-<part name="R1" library="rcl" library_urn="urn:adsk.eagle:library:334" deviceset="R-EU_" device="0204/5" package3d_urn="urn:adsk.eagle:package:23488/1"/>
-<part name="R2" library="rcl" library_urn="urn:adsk.eagle:library:334" deviceset="R-EU_" device="0204/5" package3d_urn="urn:adsk.eagle:package:23488/1"/>
-<part name="R3" library="rcl" library_urn="urn:adsk.eagle:library:334" deviceset="R-EU_" device="0204/5" package3d_urn="urn:adsk.eagle:package:23488/1"/>
-<part name="R4" library="rcl" library_urn="urn:adsk.eagle:library:334" deviceset="R-EU_" device="0207/15" package3d_urn="urn:adsk.eagle:package:23492/1"/>
-<part name="C1" library="rcl" library_urn="urn:adsk.eagle:library:334" deviceset="C-EU" device="102-043X133" package3d_urn="urn:adsk.eagle:package:23647/1"/>
+<part name="R1" library="rcl" library_urn="urn:adsk.eagle:library:334" deviceset="R-US_" device="0207/2V" package3d_urn="urn:adsk.eagle:package:23490/1" value="1k"/>
+<part name="R2" library="rcl" library_urn="urn:adsk.eagle:library:334" deviceset="R-US_" device="0207/2V" package3d_urn="urn:adsk.eagle:package:23490/1" value="1k"/>
+<part name="R3" library="rcl" library_urn="urn:adsk.eagle:library:334" deviceset="R-EU_" device="0204/5" package3d_urn="urn:adsk.eagle:package:23488/1" value="1k"/>
+<part name="R4" library="rcl" library_urn="urn:adsk.eagle:library:334" deviceset="R-EU_" device="0207/15" package3d_urn="urn:adsk.eagle:package:23492/1" value="470"/>
+<part name="C1" library="rcl" library_urn="urn:adsk.eagle:library:334" deviceset="C-EU" device="102-043X133" package3d_urn="urn:adsk.eagle:package:23647/1" value="100nF"/>
 <part name="GND1" library="supply1" library_urn="urn:adsk.eagle:library:371" deviceset="GND" device=""/>
 <part name="+3V1" library="supply1" library_urn="urn:adsk.eagle:library:371" deviceset="+3V3" device=""/>
 <part name="GND2" library="supply1" library_urn="urn:adsk.eagle:library:371" deviceset="GND" device=""/>
-<part name="R5" library="rcl" library_urn="urn:adsk.eagle:library:334" deviceset="R-EU_" device="0207/15" package3d_urn="urn:adsk.eagle:package:23492/1"/>
+<part name="R5" library="rcl" library_urn="urn:adsk.eagle:library:334" deviceset="R-EU_" device="0207/15" package3d_urn="urn:adsk.eagle:package:23492/1" value="470"/>
 <part name="+3V2" library="supply1" library_urn="urn:adsk.eagle:library:371" deviceset="+3V3" device=""/>
 <part name="GND3" library="supply1" library_urn="urn:adsk.eagle:library:371" deviceset="GND" device=""/>
@@
 <attribute name="NAME" x="-15.24" y="12.7" size="1.27" layer="94"/>
 </instance>
-<instance part="T1" gate="-1" x="137.16" y="60.96" smashed="yes" rot="R180">
-<attribute name="NAME" x="133.35" y="58.42" size="1.778" layer="95" rot="R180"/>
-<attribute name="VALUE" x="133.35" y="60.96" size="1.778" layer="96" rot="R180"/>
+<instance part="T1" gate="-1" x="137.16" y="60.96" smashed="yes" rot="MR180">
+<attribute name="NAME" x="140.97" y="58.42" size="1.778" layer="95" rot="MR180"/>
+<attribute name="VALUE" x="140.97" y="60.96" size="1.778" layer="96" rot="MR180"/>
 </instance>
 <instance part="R1" gate="G$1" x="0" y="40.64" smashed="yes">
@@
 </segment>
 </net>
-<net name="N$6" class="0">
-<segment>
-<pinref part="R4" gate="G$1" pin="2"/>
-<wire x1="124.46" y1="63.5" x2="124.46" y2="53.34" width="0.1524" layer="91"/>
-<pinref part="T1" gate="-1" pin="G"/>
-<wire x1="124.46" y1="53.34" x2="142.24" y2="53.34" width="0.1524" layer="91"/>
-<wire x1="142.24" y1="53.34" x2="142.24" y2="60.96" width="0.1524" layer="91"/>
-</segment>
-</net>
 <net name="BOMB" class="0">
 <segment>
@@
 <net name="LINE" class="0">
 <segment>
-<wire x1="134.62" y1="73.66" x2="144.78" y2="73.66" width="0.1524" layer="91"/>
 <label x="149.86" y="73.66" size="1.778" layer="95"/>
 <pinref part="T1" gate="-1" pin="A1"/>
-<wire x1="137.16" y1="63.5" x2="134.62" y2="63.5" width="0.1524" layer="91"/>
-<wire x1="134.62" y1="63.5" x2="134.62" y2="73.66" width="0.1524" layer="91"/>
-<junction x="134.62" y="73.66"/>
+<wire x1="137.16" y1="73.66" x2="144.78" y2="73.66" width="0.1524" layer="91"/>
 <pinref part="C1" gate="G$1" pin="2"/>
 <wire x1="126.492" y1="73.406" x2="126.492" y2="73.66" width="0.1524" layer="91"/>
-<wire x1="126.492" y1="73.66" x2="134.62" y2="73.66" width="0.1524" layer="91"/>
+<wire x1="126.492" y1="73.66" x2="137.16" y2="73.66" width="0.1524" layer="91"/>
+<wire x1="137.16" y1="63.5" x2="137.16" y2="73.66" width="0.1524" layer="91"/>
+<junction x="137.16" y="73.66"/>
 </segment>
 <segment>
@@
 </segment>
 </net>
+<net name="N$6" class="0">
+<segment>
+<pinref part="R4" gate="G$1" pin="2"/>
+<pinref part="T1" gate="-1" pin="G"/>
+<wire x1="124.46" y1="63.5" x2="132.08" y2="63.5" width="0.1524" layer="91"/>
+<wire x1="132.08" y1="63.5" x2="132.08" y2="60.96" width="0.1524" layer="91"/>
+</segment>
+</net>

Commit message: up2
Connections:
- removed net N$2: R1.2, SV1.6
- net TRIAC: now also R1.2, SV1.6
Changed lines of the file:
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@@
 </busses>
 <nets>
-<net name="N$2" class="0">
-<segment>
-<wire x1="12.7" y1="40.64" x2="12.7" y2="58.42" width="0.1524" layer="91"/>
-<pinref part="SV1" gate="G$1" pin="6"/>
-<wire x1="12.7" y1="58.42" x2="7.62" y2="58.42" width="0.1524" layer="91"/>
-<pinref part="R1" gate="G$1" pin="2"/>
-<wire x1="5.08" y1="40.64" x2="12.7" y2="40.64" width="0.1524" layer="91"/>
-</segment>
-</net>
 <net name="N$3" class="0">
 <segment>
@@
 <label x="53.34" y="73.66" size="1.778" layer="95"/>
 </segment>
+<segment>
+<wire x1="12.7" y1="40.64" x2="12.7" y2="58.42" width="0.1524" layer="91"/>
+<pinref part="SV1" gate="G$1" pin="6"/>
+<wire x1="12.7" y1="58.42" x2="7.62" y2="58.42" width="0.1524" layer="91"/>
+<pinref part="R1" gate="G$1" pin="2"/>
+<wire x1="5.08" y1="40.64" x2="12.7" y2="40.64" width="0.1524" layer="91"/>
+<wire x1="12.7" y1="40.64" x2="25.4" y2="40.64" width="0.1524" layer="91"/>
+<junction x="12.7" y="40.64"/>
+<label x="27.94" y="40.64" size="1.778" layer="95"/>
+</segment>
 </net>
